File: board/pico-logic-analyzer.kicad_pcb (KiCad board)
At the start: 4 copper layers, 85 x 57.5 mm, 67 parts, among them J1 Conn_02x03_Odd_Even, J10 Conn_02x03_Odd_Even, J11 Conn_01x01, J2 Conn_02x03_Odd_Even, J3 Conn_02x03_Odd_Even, J4 Conn_02x03_Odd_Even, J5 Conn_02x03_Odd_Even, J6 Conn_02x03_Odd_Even, J7 Conn_02x03_Odd_Even, J8 Conn_02x03_Odd_Even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

Commit message: added export script
Other:
- board text added: "git commit GITHASH"

Commit message: update templating to do date and user-defined version number instead of trying to make commit hash work
also, will need to revisit the timestamps that are being generated on otherwise identical gerbers
Other:
- board text added: "REV _RV DEV MON_DD_YYYY"
- board text removed: "REV 1 DEV Nov 28 2024"
- board text removed: "git commit GITHASH"
Changed lines of the file:
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@@
 		)
 	)
-	(gr_text "REV 1 DEV\nNov 28 2024"
+	(gr_text "REV _RV DEV\nMON_DD_YYYY"
 		(at 153.75 109.25 0)
 		(layer "B.SilkS")
@@
 		)
 	)
-	(gr_text "git commit GITHASH"
-		(at 194.75 109 0)
-		(layer "F.SilkS")
-		(effects
-			(font
-				(size 0.75 0.75)
-				(thickness 0.15)
-				(bold yes)
-			)
-			(justify right bottom)
-		)
-	)
 	(gr_text "PULLDOWN"
 		(at 141.75 103.75 0)
@@
 		)
 	)
-	(gr_text "REV 1 DEV\nNov 28 2024"
+	(gr_text "REV _RV DEV\nMON_DD_YYYY"
 		(at 133.25 109.25 0)
 		(layer "F.SilkS")
