File: buffer.kicad_sch (KiCad schematic)
At the start: 10 parts, among them J5 Conn_02x03_Odd_Even, J7 Conn_02x03_Odd_Even, SW3 SW_DIP_x04, U4 TXB0104PW (fit with U104)

Commit message: new project structure
Other:
- note added: "${PROJECTNAME}"
- note added: "${PROJECT_GIT} ${GIT_SHORTHASH} ${AUTHOR}"
- note added: "(sch) ${SCH_REV_DATE}"
- note added: "(sch) ${SCH_REV}"
- note added: "Pico Logic Analyzer- Digital Block"
Changed lines of the file:
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@@
 	(generator_version "9.0")
 	(paper "A4")
+	(text "${PROJECTNAME}"
+		(exclude_from_sim no)
+		(at 186.436 190.246 0)
+		(effects
+			(font
+				(size 1.27 1.27)
+			)
+			(justify left bottom)
+		)
+	)
+	(text "${PROJECT_GIT}\n${GIT_SHORTHASH}\n${AUTHOR}"
+		(exclude_from_sim no)
+		(at 285.242 181.864 0)
+		(effects
+			(font
+				(size 1.27 1.27)
+			)
+			(justify right top)
+		)
+	)
+	(text "(sch) ${SCH_REV}"
+		(exclude_from_sim no)
+		(at 268.478 193.802 0)
+		(effects
+			(font
+				(size 1.27 1.27)
+			)
+			(justify left bottom)
+		)
+	)
+	(text "(sch) ${SCH_REV_DATE}"
+		(exclude_from_sim no)
+		(at 206.502 193.802 0)
+		(effects
+			(font
+				(size 1.27 1.27)
+			)
+			(justify left bottom)
+		)
+	)
 	(text "This component is intended for PIN JUMPERS!"
 		(exclude_from_sim no)
@@
 		)
 	)
+	(text "Pico Logic Analyzer- Digital Block"
+		(exclude_from_sim no)
+		(at 177.038 166.624 0)
+		(effects
+			(font
+				(size 3.81 3.81)
+			)
+			(justify left top)
+		)
+	)
