File: pico-logic-analyzer.kicad_pcb (KiCad board)
At the start: 4 copper layers, 57.5 x 57.5 mm, 47 parts, among them J1 Conn_02x03_Odd_Even, J2 Conn_02x03_Odd_Even, J3 Conn_02x03_Odd_Even, J4 Conn_02x03_Odd_Even, J5 Conn_02x03_Odd_Even, J6 Conn_02x03_Odd_Even, J7 Conn_02x03_Odd_Even, J8 Conn_01x01, SW1 SW_DIP_x04, SW2 SW_Push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

Commit message: new project structure
Parts:
- added G1: oshw!, Symbol:OSHW-Logo2_7.3x6mm_SilkScreen, B.Cu at (101.0, 79.5)
Other:
- board text added: "${AUTHOR} ${PROJECT_GIT} commit ${GIT_SHORTHASH}"
- board text added: "${PROJECTNAME}"
- board text added: "${PROJECT_GIT} ${GIT_SHORTHASH} ${AUTHOR}"
- board text added: "(board) ${BOARD_REV_DATE}"
- board text added: "(board) ${BOARD_REV}"
- board text added: "RPi Pico Logic Analyzer Carrier"
- board text added: "board rev ${BOARD_REV} ${BOARD_REV_DATE}"
- board text added: "designed for github.com/pico-coder/sigrok-pico/ firmware"
- board text removed: "<3 from Asa Anderson github.com/tandej/pico-logic-analyzer github.com/pico-coder/sigrok-pico"
- board text removed: "JLCJLCJLCJLC"
- board text removed: "PICO-LA-CARRIER"
- board text removed: "REV _RV DEV MON_DD_YYYY"
