File: pico-logic-analyzer.kicad_sch (KiCad schematic)
At the start: 17 parts, among them J2 Conn_02x03_Odd_Even, J8 Conn_01x01, SW2 SW_Push, U2 LM4040DBZ-5, U3 LM2665M6

Commit message: new project structure
Other:
- note added: "${PROJECTNAME}"
- note added: "${PROJECT_GIT} ${GIT_SHORTHASH} ${AUTHOR}"
- note added: "(sch) ${SCH_REV_DATE}"
- note added: "(sch) ${SCH_REV}"
- note added: "Pico Logic Analyzer- Top Level"
Changed lines of the file:
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@@
 	(generator_version "9.0")
 	(paper "A4")
+	(text "${PROJECTNAME}"
+		(exclude_from_sim no)
+		(at 186.182 190.5 0)
+		(effects
+			(font
+				(size 1.27 1.27)
+			)
+			(justify left bottom)
+		)
+	)
+	(text "(sch) ${SCH_REV_DATE}"
+		(exclude_from_sim no)
+		(at 206.248 194.056 0)
+		(effects
+			(font
+				(size 1.27 1.27)
+			)
+			(justify left bottom)
+		)
+	)
 	(text "Worst-case power dissipation is when load on \n1.8v is maxxed and everything else is ~0mA.\nVoltage drop ~= 100 mV, I = 12.1 mA,\nP ~= 78 mW"
 		(exclude_from_sim no)
@@
 			)
 			(justify top)
+		)
+	)
+	(text "(sch) ${SCH_REV}"
+		(exclude_from_sim no)
+		(at 268.224 194.056 0)
+		(effects
+			(font
+				(size 1.27 1.27)
+			)
+			(justify left bottom)
 		)
 	)
@@
 		)
 	)
+	(text "${PROJECT_GIT}\n${GIT_SHORTHASH}\n${AUTHOR}"
+		(exclude_from_sim no)
+		(at 284.988 182.118 0)
+		(effects
+			(font
+				(size 1.27 1.27)
+			)
+			(justify right top)
+		)
+	)
+	(text "Pico Logic Analyzer- Top Level"
+		(exclude_from_sim no)
+		(at 176.784 166.878 0)
+		(effects
+			(font
+				(size 3.81 3.81)
+			)
+			(justify left top)
+		)
+	)
